File: motordriver/driver/driverproduction1.0/driverproduction1.0.kicad_sch (KiCad schematic)
At the start: 0 parts

Commit message: 3 hours
Other:
- added sheet Line filter (emiline.kicad_sch)
- added sheet halfbridge (halfbridge.kicad_sch)

Commit message: esp32 routin
Other:
- added sheet ESP32 (espmisc.kicad_sch)
Changed lines of the file:
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@@
 (kicad_sch (version 20230121) (generator eeschema)
   (paper "A4")
+  (sheet (at 74.93 60.96) (size 40.64 31.75) (fields_autoplaced)
+    (stroke (width 0.1524) (type solid))
+    (fill (color 0 0 0 0.0000))
+    (property "Sheetname" "ESP32" (at 74.93 60.2484 0)
+      (effects (font (size 1.27 1.27)) (justify left bottom))
+    )
+    (property "Sheetfile" "espmisc.kicad_sch" (at 74.93 93.2946 0)
+      (effects (font (size 1.27 1.27)) (justify left top))
+    )
+    (instances
+      (project "driverproduction1.0"
+        (path "/80da6768-12ef-453d-855e-7545e891c31c" (page "7"))
+      )
+    )
+  )
   (sheet (at 167.64 16.51) (size 45.72 36.83) (fields_autoplaced)
     (stroke (width 0.1524) (type solid))
