File: motordriver/driver/driverproduction1.0/untitled.kicad_sch (KiCad schematic)
At the start: 34 parts, among them T230:? Transformer_1P_1S

Commit message: larp
Parts:
- added R6, R7: R, symbol Device:R
Connections:
- net at D?.1 (K), R?.1, R?.2: now also R7.1; no longer Q?.3 (S), R?.2
- net at D?.1 (K), R?.1, R?.2: now also R6.2; no longer Q?.3 (S), R?.2
- new net: Q?.3 (S), R6.1, R?.2
- new net: Q?.3 (S), R7.2, R?.2
Changed lines of the file:
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@@
   (junction (at 147.32 96.52) (diameter 0) (color 0 0 0 0)
   )
+  (junction (at 179.07 110.49) (diameter 0) (color 0 0 0 0)
+  )
+  (junction (at 228.6 91.44) (diameter 0) (color 0 0 0 0)
+  )
+  (junction (at 166.37 80.01) (diameter 0) (color 0 0 0 0)
+  )
+  (junction (at 218.44 91.44) (diameter 0) (color 0 0 0 0)
+  )
+  (junction (at 147.32 86.36) (diameter 0) (color 0 0 0 0)
+  )
+  (junction (at 158.75 93.98) (diameter 0) (color 0 0 0 0)
+  )
+  (junction (at 140.97 91.44) (diameter 0) (color 0 0 0 0)
+  )
+  (junction (at 140.97 99.06) (diameter 0) (color 0 0 0 0)
+  )
+  (junction (at 137.16 86.36) (diameter 0) (color 0 0 0 0)
+  )
+  (junction (at 109.22 93.98) (diameter 0) (color 0 0 0 0)
+  )
+  (junction (at 109.22 88.9) (diameter 0) (color 0 0 0 0)
+  )
+  (junction (at 199.39 91.44) (diameter 0) (color 0 0 0 0)
+  )
+  (junction (at 179.07 72.39) (diameter 0) (color 0 0 0 0)
+  )
+  (junction (at 185.42 102.87) (diameter 0) (color 0 0 0 0)
+  )
+  (junction (at 67.31 87.63) (diameter 0) (color 0 0 0 0)
+  )
+  (junction (at 207.01 91.44) (diameter 0) (color 0 0 0 0)
+  )
   (junction (at 161.29 80.01) (diameter 0) (color 0 0 0 0)
   )
-  (junction (at 179.07 110.49) (diameter 0) (color 0 0 0 0)
-  )
-  (junction (at 228.6 91.44) (diameter 0) (color 0 0 0 0)
-  )
-  (junction (at 166.37 80.01) (diameter 0) (color 0 0 0 0)
-  )
-  (junction (at 218.44 91.44) (diameter 0) (color 0 0 0 0)
-  )
-  (junction (at 147.32 86.36) (diameter 0) (color 0 0 0 0)
-  )
-  (junction (at 158.75 93.98) (diameter 0) (color 0 0 0 0)
-  )
-  (junction (at 140.97 91.44) (diameter 0) (color 0 0 0 0)
-  )
-  (junction (at 140.97 99.06) (diameter 0) (color 0 0 0 0)
-  )
-  (junction (at 137.16 86.36) (diameter 0) (color 0 0 0 0)
-  )
-  (junction (at 109.22 93.98) (diameter 0) (color 0 0 0 0)
-  )
-  (junction (at 109.22 88.9) (diameter 0) (color 0 0 0 0)
-  )
-  (junction (at 199.39 91.44) (diameter 0) (color 0 0 0 0)
-  )
-  (junction (at 179.07 72.39) (diameter 0) (color 0 0 0 0)
-  )
-  (junction (at 185.42 102.87) (diameter 0) (color 0 0 0 0)
-  )
-  (junction (at 67.31 87.63) (diameter 0) (color 0 0 0 0)
-  )
-  (junction (at 207.01 91.44) (diameter 0) (color 0 0 0 0)
-  )
   (junction (at 137.16 96.52) (diameter 0) (color 0 0 0 0)
   )
+  (junction (at 175.26 87.63) (diameter 0) (color 0 0 0 0)
+  )
+  (junction (at 158.75 88.9) (diameter 0) (color 0 0 0 0)
+  )
+  (junction (at 226.06 91.44) (diameter 0) (color 0 0 0 0)
+  )
+  (junction (at 144.78 96.52) (diameter 0) (color 0 0 0 0)
+  )
+  (junction (at 149.86 93.98) (diameter 0) (color 0 0 0 0)
+  )
+  (junction (at 149.86 88.9) (diameter 0) (color 0 0 0 0)
+  )
+  (junction (at 185.42 80.01) (diameter 0) (color 0 0 0 0)
+  )
+  (junction (at 67.31 95.25) (diameter 0) (color 0 0 0 0)
+  )
   (junction (at 161.29 102.87) (diameter 0) (color 0 0 0 0)
   )
-  (junction (at 175.26 87.63) (diameter 0) (color 0 0 0 0)
-  )
-  (junction (at 158.75 88.9) (diameter 0) (color 0 0 0 0)
-  )
-  (junction (at 226.06 91.44) (diameter 0) (color 0 0 0 0)
-  )
-  (junction (at 144.78 96.52) (diameter 0) (color 0 0 0 0)
-  )
-  (junction (at 149.86 93.98) (diameter 0) (color 0 0 0 0)
-  )
-  (junction (at 149.86 88.9) (diameter 0) (color 0 0 0 0)
-  )
-  (junction (at 185.42 80.01) (diameter 0) (color 0 0 0 0)
-  )
-  (junction (at 67.31 95.25) (diameter 0) (color 0 0 0 0)
-  )
   (junction (at 140.97 83.82) (diameter 0) (color 0 0 0 0)
   )
@@
     (stroke (width 0) (type default))
   )
-  (wire (pts (xy 161.29 93.98) (xy 161.29 102.87))
-    (stroke (width 0) (type default))
-  )
   (wire (pts (xy 179.07 110.49) (xy 180.34 110.49))
     (stroke (width 0) (type default))
@@
     (stroke (width 0) (type default))
   )
+  (wire (pts (xy 161.29 87.63) (xy 161.29 88.9))
+    (stroke (width 0) (type default))
+  )
   (wire (pts (xy 147.32 86.36) (xy 149.86 86.36))
     (stroke (width 0) (type default))
@@
     (stroke (width 0) (type default))
   )
+  (wire (pts (xy 161.29 101.6) (xy 161.29 102.87))
+    (stroke (width 0) (type default))
+  )
   (wire (pts (xy 222.25 87.63) (xy 222.25 88.9))
     (stroke (width 0) (type default))
@@
   )
   (wire (pts (xy 176.53 90.17) (xy 158.75 90.17))
-    (stroke (width 0) (type default))
-  )
-  (wire (pts (xy 161.29 80.01) (xy 161.29 88.9))
     (stroke (width 0) (type default))
   )
@@
     )
   )
+  (symbol (lib_id "Device:R") (at 161.29 83.82 0) (unit 1)
+    (in_bom yes) (on_board yes) (dnp no) (fields_autoplaced)
+    (property "Reference" "R6" (at 163.83 82.55 0)
+      (effects (font (size 1.27 1.27)) (justify left))
+    )
+    (property "Value" "R" (at 163.83 85.09 0)
+      (effects (font (size 1.27 1.27)) (justify left))
+    )
+    (property "Footprint" "" (at 159.512 83.82 90)
+      (effects (font (size 1.27 1.27)) hide)
+    )
+    (property "Datasheet" "~" (at 161.29 83.82 0)
+      (effects (font (size 1.27 1.27)) hide)
+    )
+    (pin "1")
+    (pin "2")
+    (instances
+      (project "driverproduction1.0"
+        (path "/80da6768-12ef-453d-855e-7545e891c31c/ebafb242-e5ab-4243-abe4-e8fcc7c0a63e"
+          (reference "R6") (unit 1)
+        )
+      )
+    )
+  )
   (symbol (lib_id "power:GND") (at 176.53 80.01 0) (unit 1)
     (in_bom yes) (on_board yes) (dnp no) (fields_autoplaced)
@@
         )
       )
+    )
+  )
+  (symbol (lib_id "Device:R") (at 161.29 97.79 0) (unit 1)
+    (in_bom yes) (on_board yes) (dnp no) (fields_autoplaced)
+    (property "Reference" "R7" (at 163.83 96.52 0)
+      (effects (font (size 1.27 1.27)) (justify left))
+    )
+    (property "Value" "R" (at 163.83 99.06 0)
+      (effects (font (size 1.27 1.27)) (justify left))
+    )
+    (property "Footprint" "" (at 159.512 97.79 90)
+      (effects (font (size 1.27 1.27)) hide)
+    )
+    (property "Datasheet" "~" (at 161.29 97.79 0)
+      (effects (font (size 1.27 1.27)) hide)
+    )
+    (pin "1")
+    (pin "2")
+    (instances
+      (project "driverproduction1.0"
+        (path "/80da6768-12ef-453d-855e-7545e891c31c/ebafb242-e5ab-4243-abe4-e8fcc7c0a63e"
+          (reference "R7") (unit 1)
+        )
+      )
