File: motordriver/driver/driverproduction1.0/driverproduction1.0.kicad_pcb (KiCad board)
At the start: 4 copper layers, 180 x 100 mm, 86 parts

Commit message: hahhaha
Parts:
- added REF**: D_0805_2012Metric, Diode_SMD:D_0805_2012Metric, F.Cu at (168.9, 48.5)
- added REF**: R_Axial_DIN0204_L3.6mm_D1.6mm_P5.08mm_Horizontal, Resistor_THT:R_Axial_DIN0204_L3.6mm_D1.6mm_P5.08mm_Horizontal, F.Cu at (187.9, 42.7)
- added REF**: R_Axial_DIN0204_L3.6mm_D1.6mm_P5.08mm_Horizontal, Resistor_THT:R_Axial_DIN0204_L3.6mm_D1.6mm_P5.08mm_Horizontal, F.Cu at (184.9, 46.1)
- added REF**: R_Axial_DIN0204_L3.6mm_D1.6mm_P5.08mm_Horizontal, Resistor_THT:R_Axial_DIN0204_L3.6mm_D1.6mm_P5.08mm_Horizontal, F.Cu at (196.5, 45.7)
- added REF**: D_0805_2012Metric, Diode_SMD:D_0805_2012Metric, F.Cu at (169.8, 41.5)
- added REF**: R_Axial_DIN0204_L3.6mm_D1.6mm_P5.08mm_Horizontal, Resistor_THT:R_Axial_DIN0204_L3.6mm_D1.6mm_P5.08mm_Horizontal, F.Cu at (192.9, 62.2)
- moved REF** 14.9 mm to (167.0, 29.8)
- moved REF** 14.0 mm to (167.8, 62.7)
- moved IRLU014PBF 11.4 mm to (190.6, 53.3), turned to 90 degrees
- moved IRLU014PBF 0.96 mm to (194.2, 37.4)
Routing:
- net (no net): track 1383.2 -> 1756.3 mm, vias 45 -> 46

Commit message: almost there!
Parts:
- removed the REF** at (61.3, 81.9)
- removed the REF** at (68.4, 87.9)
- removed the REF** at (70.8, 86.5)
- removed the REF** at (61.3, 82.7)
- removed the REF** at (70.0, 87.9)
- removed the REF** at (69.2, 86.5)
- added REF**: R_0402_1005Metric, Resistor_SMD:R_0402_1005Metric, F.Cu at (63.7, 87.3)
- added REF**: C_0201_0603Metric, Capacitor_SMD:C_0201_0603Metric, F.Cu at (54.5, 90.0)
- added REF**: C_0201_0603Metric, Capacitor_SMD:C_0201_0603Metric, F.Cu at (76.3, 87.5)
- added REF**: C_0201_0603Metric, Capacitor_SMD:C_0201_0603Metric, F.Cu at (76.3, 88.7)
- added REF**: C_0201_0603Metric, Capacitor_SMD:C_0201_0603Metric, F.Cu at (77.9, 88.7)
- added REF**: C_0201_0603Metric, Capacitor_SMD:C_0201_0603Metric, F.Cu at (52.9, 88.2)
- added REF**: C_0201_0603Metric, Capacitor_SMD:C_0201_0603Metric, F.Cu at (77.9, 87.5)
- added REF**: R_0402_1005Metric, Resistor_SMD:R_0402_1005Metric, F.Cu at (62.2, 87.0)
- added REF**: C_0201_0603Metric, Capacitor_SMD:C_0201_0603Metric, F.Cu at (54.5, 90.8)
- added REF**: C_0201_0603Metric, Capacitor_SMD:C_0201_0603Metric, F.Cu at (52.6, 90.0)
- added REF**: C_0402_1005Metric, Capacitor_SMD:C_0402_1005Metric, F.Cu at (71.8, 103.7)
- added REF**: C_0201_0603Metric, Capacitor_SMD:C_0201_0603Metric, F.Cu at (107.6, 180.1)
- added REF**: C_0402_1005Metric, Capacitor_SMD:C_0402_1005Metric, F.Cu at (57.8, 77.0)
- added REF**: C_0402_1005Metric, Capacitor_SMD:C_0402_1005Metric, F.Cu at (53.6, 77.0)
- added REF**: C_0201_0603Metric, Capacitor_SMD:C_0201_0603Metric, F.Cu at (59.7, 80.5)
- added REF**: C_0201_0603Metric, Capacitor_SMD:C_0201_0603Metric, F.Cu at (54.5, 89.2)
- added REF**: R_0402_1005Metric, Resistor_SMD:R_0402_1005Metric, F.Cu at (65.9, 85.2)
- added REF**: C_0201_0603Metric, Capacitor_SMD:C_0201_0603Metric, F.Cu at (0.00, 0.00)
- moved  AD5141WBCPZ10-RL7 8.27 mm to (71.4, 85.5)
- moved REF** 2.01 mm to (58.2, 88.1)
Routing:
- net (no net): track 1756.3 -> 2210.7 mm, vias 46 -> 64

Commit message: almost!!
Parts:
- added REF**: Crystal_SMD_3225-4Pin_3.2x2.5mm, Crystal:Crystal_SMD_3225-4Pin_3.2x2.5mm, F.Cu at (76.3, 96.3)
- added REF**: C_0201_0603Metric, Capacitor_SMD:C_0201_0603Metric, F.Cu at (68.1, 88.6)
- added REF**: C_0201_0603Metric, Capacitor_SMD:C_0201_0603Metric, F.Cu at (68.1, 87.8)
- added REF**: C_0402_1005Metric, Capacitor_SMD:C_0402_1005Metric, F.Cu at (59.1, 90.9)
- added REF**: C_0402_1005Metric, Capacitor_SMD:C_0402_1005Metric, F.Cu at (60.2, 91.5)
- added REF**: R_0402_1005Metric, Resistor_SMD:R_0402_1005Metric, F.Cu at (57.0, 92.5)
Routing:
- net (no net): track 2210.7 -> 2323.0 mm, vias 64 -> 75

Commit message: just need to do the final touches now!
Parts:
- added REF**: R_0402_1005Metric, Resistor_SMD:R_0402_1005Metric, F.Cu at (76.8, 98.6)
- added REF**: PinHeader_1x16_P1.00mm_Vertical, Connector_PinHeader_1.00mm:PinHeader_1x16_P1.00mm_Vertical, F.Cu at (164.8, 112.8)
- added REF**: PinHeader_1x01_P1.00mm_Vertical, Connector_PinHeader_1.00mm:PinHeader_1x01_P1.00mm_Vertical, F.Cu at (147.7, 94.7)
- added REF**: D_DO-15_P5.08mm_Vertical_AnodeUp, Diode_THT:D_DO-15_P5.08mm_Vertical_AnodeUp, B.Cu at (151.4, 99.3)
- added REF**: C_0402_1005Metric, Capacitor_SMD:C_0402_1005Metric, F.Cu at (76.4, 93.2)
- added REF**: PinHeader_1x06_P1.00mm_Vertical, Connector_PinHeader_1.00mm:PinHeader_1x06_P1.00mm_Vertical, F.Cu at (73.7, 91.8)
- added REF**: PinHeader_1x10_P1.00mm_Vertical, Connector_PinHeader_1.00mm:PinHeader_1x10_P1.00mm_Vertical, F.Cu at (116.0, 103.3)
- added REF**: C_0402_1005Metric, Capacitor_SMD:C_0402_1005Metric, F.Cu at (80.2, 98.4)
- added REF**: PinHeader_1x16_P1.00mm_Vertical, Connector_PinHeader_1.00mm:PinHeader_1x16_P1.00mm_Vertical, F.Cu at (157.8, 114.0)
- added REF**: PinHeader_1x01_P1.00mm_Vertical, Connector_PinHeader_1.00mm:PinHeader_1x01_P1.00mm_Vertical, F.Cu at (144.1, 93.7)
- added REF**: C_0201_0603Metric, Capacitor_SMD:C_0201_0603Metric, F.Cu at (63.5, 91.4)
- added REF**: PinHeader_1x01_P1.00mm_Vertical, Connector_PinHeader_1.00mm:PinHeader_1x01_P1.00mm_Vertical, F.Cu at (119.4, 111.8)
- added REF**: C_0201_0603Metric, Capacitor_SMD:C_0201_0603Metric, F.Cu at (59.6, 100.0)
- added REF**: PinHeader_1x16_P1.00mm_Vertical, Connector_PinHeader_1.00mm:PinHeader_1x16_P1.00mm_Vertical, F.Cu at (60.0, 110.9)
- moved REF** 3.67 mm to (79.6, 94.7), turned to 90 degrees
Routing:
- net (no net): track 2323.0 -> 2736.9 mm, vias 75 -> 85

Commit message: to messy
Parts:
- removed the REF** at (76.8, 98.6)
- removed the REF** at (57.0, 92.5)
- removed the REF** at (79.6, 94.7)
- removed the REF** at (63.7, 87.3)
- removed the REF** at (76.4, 93.2)
- removed the REF** at (73.7, 91.8)
- removed the REF** at (80.2, 98.4)
- removed the REF** at (76.3, 87.5)
- removed the REF** at (77.9, 88.7)
- removed the REF** at (157.8, 114.0)
- removed the REF** at (76.3, 88.7)
- removed the REF** at (63.5, 91.4)
- removed the REF** at (68.1, 88.6)
- removed the REF** at (77.9, 87.5)
- removed the REF** at (59.6, 100.0)
- removed the REF** at (62.2, 87.0)
- removed the REF** at (60.0, 110.9)
- removed the REF** at (71.8, 103.7)
- removed the REF** at (68.1, 87.8)
- removed the REF** at (65.9, 85.2)
- removed the REF** at (59.1, 90.9)
- removed the REF** at (60.2, 91.5)
- moved REF** 12.4 mm to (77.0, 103.6)
- moved REF** 8.78 mm to (66.6, 90.7)
- moved  AD5141WBCPZ10-RL7 7.75 mm to (75.8, 91.8)
- moved REF** 7.36 mm to (60.7, 78.9)
- moved REF** 7.36 mm to (62.8, 83.1)
- moved REF** 7.36 mm to (64.8, 78.9)
- moved REF** 7.36 mm to (66.8, 82.5)
Routing:
- net (no net): track 2736.9 -> 2106.3 mm, vias 85 -> 49

Commit message: 3
Parts:
- added REF**: C_0603_1608Metric, Capacitor_SMD:C_0603_1608Metric, F.Cu at (94.6, 96.2)
- added REF**: C_0603_1608Metric, Capacitor_SMD:C_0603_1608Metric, F.Cu at (99.1, 96.2)
- added REF**: C_0402_1005Metric, Capacitor_SMD:C_0402_1005Metric, F.Cu at (92.7, 95.7)
- added REF**: C_0603_1608Metric, Capacitor_SMD:C_0603_1608Metric, F.Cu at (96.9, 96.2)
Routing:
- net (no net): track 2106.3 -> 2147.3 mm, vias 49 -> 51

Commit message: test
Parts:
- added REF**: R_0603_1608Metric, Resistor_SMD:R_0603_1608Metric, F.Cu at (60.9, 93.6)
- added REF**: C_0201_0603Metric, Capacitor_SMD:C_0201_0603Metric, F.Cu at (80.2, 90.1)
- added REF**: C_0402_1005Metric, Capacitor_SMD:C_0402_1005Metric, B.Cu at (66.7, 87.3)
- added REF**: R_Axial_DIN0204_L3.6mm_D1.6mm_P2.54mm_Vertical, Resistor_THT:R_Axial_DIN0204_L3.6mm_D1.6mm_P2.54mm_Vertical, F.Cu at (57.0, 91.2)
- added REF**: PinHeader_1x08_P1.00mm_Vertical, Connector_PinHeader_1.00mm:PinHeader_1x08_P1.00mm_Vertical, F.Cu at (73.3, 114.4)
- added REF**: C_0201_0603Metric, Capacitor_SMD:C_0201_0603Metric, F.Cu at (79.9, 110.4)
- added REF**: C_0402_1005Metric, Capacitor_SMD:C_0402_1005Metric, F.Cu at (67.6, 93.9)
- added REF**: C_0201_0603Metric, Capacitor_SMD:C_0201_0603Metric, F.Cu at (70.6, 107.8)
- added REF**: C_0201_0603Metric, Capacitor_SMD:C_0201_0603Metric, F.Cu at (73.8, 91.6)
- added REF**: C_0201_0603Metric, Capacitor_SMD:C_0201_0603Metric, F.Cu at (81.1, 89.4)
- added REF**: C_0201_0603Metric, Capacitor_SMD:C_0201_0603Metric, F.Cu at (66.1, 88.5)
- added REF**: C_0201_0603Metric, Capacitor_SMD:C_0201_0603Metric, F.Cu at (81.9, 90.1)
- added REF**: C_0201_0603Metric, Capacitor_SMD:C_0201_0603Metric, F.Cu at (67.0, 94.8)
- added REF**: C_0201_0603Metric, Capacitor_SMD:C_0201_0603Metric, F.Cu at (72.7, 92.0)
- added REF**: C_0201_0603Metric, Capacitor_SMD:C_0201_0603Metric, F.Cu at (73.9, 96.9)
- added REF**: R_0603_1608Metric, Resistor_SMD:R_0603_1608Metric, F.Cu at (70.5, 85.6)
- added REF**: C_0201_0603Metric, Capacitor_SMD:C_0201_0603Metric, F.Cu at (76.9, 97.0)
- added REF**: R_0402_1005Metric, Resistor_SMD:R_0402_1005Metric, F.Cu at (57.5, 94.1)
- added REF**: C_0201_0603Metric, Capacitor_SMD:C_0201_0603Metric, F.Cu at (79.4, 89.4)
- REF**: moved to F.Cu
- moved REF** 8.23 mm to (111.5, 114.1)
- moved REF** 7.61 mm to (108.4, 103.4)
- moved  AD5141WBCPZ10-RL7 2.93 mm to (75.2, 89.0)
- moved REF** 1.67 mm to (65.1, 91.2)
Routing:
- net (no net): track 2147.3 -> 2742.1 mm, vias 51 -> 84
